File: MiniRoverPowerBoard_Hardware/MiniRoverPowerBoard_Hardware.sch (KiCad schematic (older format))
At the start: 19 parts

Commit message: Finished Power Control, Started uC
Parts:
- removed C?: C_Small, symbol Device:C_Small
- removed D?: D_Zener, symbol Device:D_Zener
- removed R? (x2): R_Small, symbol Device:R_Small
- added B?: Buzzer, symbol MRDT_Devices:Buzzer
- added C?: 1n, symbol Device:C_Small
- added D?: 3V3_Zener, symbol Device:D_Zener
- added R? (x2): 20k, symbol Device:R_Small
- added R? (x2): 13k, symbol Device:R_Small
- added U?: ACS722xLCTR-40AU, Package_SO:SOIC-8_3.9x4.9mm_P1.27mm, symbol Sensor_Current:ACS722xLCTR-40AU
- added U?: ARDUINO_MICRO_SHIELD, symbol MiniRoverPowerBoard_Hardware:ARDUINO_MICRO_SHIELD
Connections:
- net labels added: 3V3_PWR, LOG_SW_EN, PACK_IMEAS, V_LOG_SENSE
- wire segments 59 -> 83
Other:
- note added: "Current\nMeasurment"
- note added: "E-Stop"
- note added: "Input"
- note added: "Logic Power Switch"
- note added: "Microcontroller"
- note added: "Output"
- note added: "Power Control"

Commit message: Added motor drivers, 3v3 buck, sw, uC assignments
Next is to add remote control
Parts:
- added C? (x3): 10u, symbol Device:C_Small
- added C? (x2): 470u, Capacitor_THT:CP_Radial_D8.0mm_P3.50mm, symbol Device:CP1_Small
- added Conn? (x4): AndersonPP, symbol MRDT_Connectors:AndersonPP
- added D? (x7): LED, symbol Device:LED
- added D?: D_Schottky, Diode_SMD:D_0603_1608Metric_Pad1.05x0.95mm_HandSolder, symbol Device:D_Schottky_Small
- added L?: 47uH, Capacitor_THT:CP_Radial_D5.0mm_P2.00mm, symbol pspice:INDUCTOR
- added Q?: Q_NMOS_GSD, symbol Device:Q_NMOS_GSD
- added R? (x4): 10k, symbol Device:R_Small
- added R? (x6): 510, symbol Device:R_Small
- added R?: 100, symbol Device:R_Small
- added R? (x6): 1k, symbol Device:R_Small
- added SW?: SW_SPDT, symbol Switch:SW_SPDT
- added SW? (x2): SW_Push, symbol Switch:SW_Push
- added U? (x2): VNH5019A_E, symbol MRDT_ICs:VNH5019A_E
- added U?: AP1509, symbol MRDT_ICs:AP1509
Connections:
- net labels added: +3V3, +5V, BUZZER_EN, DIRECTION_SW, IN_A1, IN_A2, IN_B1, IN_B2, LEFT_PWM, LEFT_SW, OUT_A_LEFT, OUT_A_RIGHT, OUT_B_LEFT, OUT_B_RIGHT, RIGHT_PWM, RIGHT_SW
- net labels removed: 3V3_PWR
- wire segments 83 -> 293
- no-connect marks 0 -> 5
Other:
- note added: "10mA"
- note added: "13mA"
- note added: "16mA"
- note added: "3V3 Regulation"
- note added: "500mA limit due to Inductor"
- note added: "8.4V Max\n7.4V Nominal\n5.0V Min (Broken)"
- note added: "8.4V to 3.3V"
- note added: "Buzzer"
- note added: "Drive Switches"
- note added: "Green"
- note added: "Indication"
- note added: "Left Motors"
- note added: "Motor Drivers"
- note added: "Orange"
- note added: "Right Motors"

Commit message: Added Controller Conn and Pins on uC
Parts:
- added C? (x2): 10u, symbol Device:C_Small
- added Conn?: Molex_SL_07, symbol MRDT_Connectors:Molex_SL_07
- added D?: D_Schottky, Diode_SMD:D_0603_1608Metric_Pad1.05x0.95mm_HandSolder, symbol Device:D_Schottky_Small
- added L?: 47uH, Capacitor_THT:CP_Radial_D5.0mm_P2.00mm, symbol pspice:INDUCTOR
- added U?: AP1509, symbol MRDT_ICs:AP1509
Connections:
- net labels added: CONTROLLER_ATT, CONTROLLER_CLK, CONTROLLER_CMD, CONTROLLER_DAT
- wire segments 293 -> 336
- no-connect marks 5 -> 16
Other:
- note added: "5V Regulation"
- note added: "Controller Conn"
- note added: "Min Input Volatge: 6V"
- note added: "Min Input Voltage for each: 4.5V\n500mA limit each due to inductors"
- note removed: "500mA limit due to Inductor"

Commit message: Footprints assigned to symbols; Netlist generated
Parts:
- removed Q?: Q_PMOS_GDS, symbol Device:Q_PMOS_GDS
- added Q3: Q_PMOS_GDS, Package_TO_SOT_SMD:TO-252-2, symbol Device:Q_PMOS_GDS
- B1: renamed from B?; footprint (none) -> MRDT_Devices:BUZZER_SMI_1324_TW_5V_2_R
- C1, C2, C3, C4, C7, C8: renamed from C?; footprint (none) -> Capacitor_SMD:C_0603_1608Metric_Pad1.05x0.95mm_HandSolder
- Conn1, Conn2, Conn3, Conn4: renamed from Conn?; footprint (none) -> MRDT_Connectors:Anderson_2_Horizontal_Side_by_Side
- Conn5: renamed from Conn?; footprint (none) -> MRDT_Connectors:MOLEX_SL_02_Vertical
- Conn6: renamed from Conn?; footprint (none) -> MRDT_Connectors:MOLEX_SL_07_Vertical
- D1, D9: renamed from D?; footprint (none) -> Diode_SMD:D_SOD-123
- D10, D11, D2, D3, D4, D5, D6: renamed from D?; footprint (none) -> LED_SMD:LED_0603_1608Metric_Pad1.05x0.95mm_HandSolder
- F1: renamed from F?; footprint (none) -> MRDT_Passives:ATC_Fuse_Block
- Q1, Q2, Q4: renamed from Q?; footprint (none) -> Package_TO_SOT_SMD:SOT-323_SC-70_Handsoldering
- R1, R10, R13, R14, R15, R16, R17, R18, R19, R2, R20, R21, R22, R23, R24, R25, R3, R4, R5, R6, R7, R8, R9: renamed from R?; footprint (none) -> Resistor_SMD:R_0603_1608Metric_Pad1.05x0.95mm_HandSolder
- R11: renamed from R?; value R_Small -> 30k; footprint (none) -> Resistor_SMD:R_0603_1608Metric_Pad1.05x0.95mm_HandSolder
- R12: renamed from R?; value R_Small -> 13k; footprint (none) -> Resistor_SMD:R_0603_1608Metric_Pad1.05x0.95mm_HandSolder
- SW1: renamed from SW?; footprint (none) -> MRDT_Connectors:MOLEX_SL_04_Vertical
- SW2, SW3: renamed from SW?; footprint (none) -> Button_Switch_SMD:SW_SPST_TL3305A
- SW4: renamed from SW?; footprint (none) -> Button_Switch_THT:SW_CW_GPTS203211B
- U1, U2: renamed from U?; footprint (none) -> MRDT_ICs:MultiPowerSO_30
- U4, U5: renamed from U?; footprint (none) -> Package_SO:SOIC-8_3.9x4.9mm_P1.27mm
- U6: renamed from U?; footprint (none) -> MiniRoverPowerBoard_Hardware:ARDUINO_MICRO_SHIELD
- gave numbers to parts that had none: 7

Commit message: All footprints correct and layout started
Parts:
- SW4: footprint Button_Switch_THT:SW_CW_GPTS203211B -> Button_Switch_THT:SW_CuK_OS102011MA1QN1_SPDT_Angled
- renumbered Conn1 to Conn3, Conn2 to Conn4
Connections:
- net labels added: PVDD_IN1, PVDD_IN2, PVDD_IN3
Other:
- note added: "8.4V to 2.54V\n6V to 1.81V"
Changed lines of the file:
@@
 $Comp
 L MRDT_Connectors:AndersonPP Conn1
-U 4 1 5DB30291
+U 2 1 5DB30291
 P 1200 2850
 F 0 "Conn1" H 950 2950 60  0000 C CNN
@@
 F 2 "MRDT_Connectors:Anderson_2_Horizontal_Side_by_Side" H 1050 2300 60  0001 C CNN
 F 3 "" H 1050 2300 60  0001 C CNN
-	4    1200 2850
+	2    1200 2850
 	1    0    0    -1
 $EndComp
@@
 $Comp
 L MRDT_Connectors:AndersonPP Conn2
-U 4 1 5DB3034B
+U 2 1 5DB3034B
 P 1200 3500
 F 0 "Conn2" H 950 3600 60  0000 C CNN
@@
 F 2 "MRDT_Connectors:Anderson_2_Horizontal_Side_by_Side" H 1050 2950 60  0001 C CNN
 F 3 "" H 1050 2950 60  0001 C CNN
-	4    1200 3500
+	2    1200 3500
 	1    0    0    -1
 $EndComp
@@
 F 0 "SW4" H 6150 8035 50  0000 C CNN
 F 1 "SW_SPDT" H 6150 7944 50  0000 C CNN
-F 2 "Button_Switch_THT:SW_CW_GPTS203211B" H 6150 7750 50  0001 C CNN
+F 2 "Button_Switch_THT:SW_CuK_OS102011MA1QN1_SPDT_Angled" H 6150 7750 50  0001 C CNN
 F 3 "" H 6150 7750 50  0001 C CNN
 	1    6150 7750
@@
 	3550 7350 3650 7350
 $Comp
-L MRDT_Connectors:AndersonPP Conn1
+L MRDT_Connectors:AndersonPP Conn3
 U 2 1 5DD4C020
 P 4550 6400
-F 0 "Conn1" H 4523 6447 60  0000 R CNN
+F 0 "Conn3" H 4523 6447 60  0000 R CNN
 F 1 "AndersonPP" H 4523 6553 60  0000 R CNN
 F 2 "MRDT_Connectors:Anderson_2_Horizontal_Side_by_Side" H 4400 5850 60  0001 C CNN
@@
 	3550 9750 3650 9750
 $Comp
-L MRDT_Connectors:AndersonPP Conn2
+L MRDT_Connectors:AndersonPP Conn4
 U 2 1 5DDD7FF9
 P 4550 8800
-F 0 "Conn2" H 4523 8847 60  0000 R CNN
+F 0 "Conn4" H 4523 8847 60  0000 R CNN
 F 1 "AndersonPP" H 4523 8953 60  0000 R CNN
 F 2 "MRDT_Connectors:Anderson_2_Horizontal_Side_by_Side" H 4400 8250 60  0001 C CNN
@@
 	0    1    -1   0
 $EndComp
+Text Label 1800 3100 0    50   ~ 0
+PVDD_IN1
+Text Label 2700 3100 0    50   ~ 0
+PVDD_IN2
+Text Label 3350 3100 0    50   ~ 0
+PVDD_IN3
+Text Notes 6500 3450 0    43   ~ 0
+8.4V to 2.54V\n6V to 1.81V
 $EndSCHEMATC

Commit message: Almost All Components Layed Out
Parts:
- removed R15: 10k, Resistor_SMD:R_0603_1608Metric_Pad1.05x0.95mm_HandSolder, symbol Device:R_Small
- removed SW4: SW_SPDT, Button_Switch_THT:SW_CuK_OS102011MA1QN1_SPDT_Angled, symbol Switch:SW_SPDT
- added C10, C11, C12, C9: 10u, Capacitor_SMD:C_0603_1608Metric_Pad1.05x0.95mm_HandSolder, symbol Device:C_Small
Connections:
- net labels removed: DIRECTION_SW
- wire segments 336 -> 343
- no-connect marks 16 -> 14

Commit message: All Comps Placed; Adding more though :(
Parts:
- added Conn?: Molex_SL_02, symbol MRDT_Connectors:Molex_SL_02
- added R? (x3): 0, Resistor_SMD:R_0603_1608Metric_Pad1.05x0.95mm_HandSolder, symbol Device:R_Small
Connections:
- net labels added: RX, TX
- wire segments 343 -> 355
Other:
- note added: "Serial Conn"

Commit message: Added Extra Buses & Started Polygons
Parts:
- added Conn10, Conn9: Molex_SL_04, MRDT_Connectors:MOLEX_SL_04_Horizontal, symbol MRDT_Connectors:Molex_SL_04
- added Conn8: Molex_SL_02, MRDT_Connectors:MOLEX_SL_02_Vertical, symbol MRDT_Connectors:Molex_SL_02
- Conn7: renamed from Conn?; footprint (none) -> MRDT_Connectors:MOLEX_SL_02_Vertical
- gave numbers to parts that had none: 3
Connections:
- wire segments 355 -> 371
Other:
- note added: "12V"
- note added: "5V"
- note added: "Extra Outputs"
- note added: "Sorry for these 12V connectors. Whole \nandersons for 12V extra busses on a \nmini rover are overkill. But I don't want \nto introduce a new connector outside \nour standards. So two pins on a \nMolex SL will get you 4A."
Changed lines of the file:
@@
 	7600 6500 5400 6500
 $Comp
-L MRDT_Connectors:Molex_SL_02 Conn?
+L MRDT_Connectors:Molex_SL_02 Conn7
 U 1 1 5DD732D9
 P 6750 5950
-F 0 "Conn?" H 6877 6108 60  0000 L CNN
+F 0 "Conn7" H 6877 6108 60  0000 L CNN
 F 1 "Molex_SL_02" H 6877 6002 60  0000 L CNN
-F 2 "" H 6750 5850 60  0001 C CNN
+F 2 "MRDT_Connectors:MOLEX_SL_02_Vertical" H 6750 5850 60  0001 C CNN
 F 3 "" H 6750 5850 60  0001 C CNN
 	1    6750 5950
@@
 $EndComp
 $Comp
-L Device:R_Small R?
+L Device:R_Small R15
 U 1 1 5DD73B63
 P 6150 5750
-F 0 "R?" V 6050 5700 50  0000 L CNN
+F 0 "R15" V 6050 5700 50  0000 L CNN
 F 1 "0" V 6150 5700 50  0000 L CNN
 F 2 "Resistor_SMD:R_0603_1608Metric_Pad1.05x0.95mm_HandSolder" H 6150 5750 50  0001 C CNN
@@
 $EndComp
 $Comp
-L Device:R_Small R?
+L Device:R_Small R26
 U 1 1 5DD75966
 P 6150 5950
-F 0 "R?" V 6050 5900 50  0000 L CNN
+F 0 "R26" V 6050 5900 50  0000 L CNN
 F 1 "0" V 6150 5900 50  0000 L CNN
 F 2 "Resistor_SMD:R_0603_1608Metric_Pad1.05x0.95mm_HandSolder" H 6150 5950 50  0001 C CNN
@@
 $EndComp
 $Comp
-L Device:R_Small R?
+L Device:R_Small R27
 U 1 1 5DD75A1C
 P 6350 5850
-F 0 "R?" H 6200 5850 50  0000 L CNN
+F 0 "R27" H 6200 5850 50  0000 L CNN
 F 1 "0" V 6350 5800 50  0000 L CNN
 F 2 "Resistor_SMD:R_0603_1608Metric_Pad1.05x0.95mm_HandSolder" H 6350 5850 50  0001 C CNN
@@
 Wire Wire Line
 	12250 7400 12300 7400
+$Comp
+L MRDT_Connectors:Molex_SL_02 Conn8
+U 1 1 5DD8021C
+P 12400 1900
+F 0 "Conn8" H 12527 2058 60  0000 L CNN
+F 1 "Molex_SL_02" H 12527 1952 60  0000 L CNN
+F 2 "MRDT_Connectors:MOLEX_SL_02_Vertical" H 12400 1800 60  0001 C CNN
+F 3 "" H 12400 1800 60  0001 C CNN
+	1    12400 1900
+	1    0    0    -1
+$EndComp
+$Comp
+L MRDT_Connectors:Molex_SL_04 Conn9
+U 1 1 5DD803DE
+P 12400 3300
+F 0 "Conn9" H 12527 3558 60  0000 L CNN
+F 1 "Molex_SL_04" H 12527 3452 60  0000 L CNN
+F 2 "MRDT_Connectors:MOLEX_SL_04_Horizontal" H 12400 3300 60  0001 C CNN
+F 3 "" H 12400 3300 60  0001 C CNN
+	1    12400 3300
+	1    0    0    -1
+$EndComp
+Text GLabel 12150 2950 0    50   Input ~ 0
+ACT_PWR
+Text GLabel 12150 3050 0    50   Input ~ 0
+ACT_PWR
+$Comp
+L power:GND #PWR0113
+U 1 1 5DD81AC3
+P 12150 3300
+F 0 "#PWR0113" H 12150 3050 50  0001 C CNN
+F 1 "GND" H 12155 3127 50  0000 C CNN
+F 2 "" H 12150 3300 50  0001 C CNN
+F 3 "" H 12150 3300 50  0001 C CNN
+	1    12150 3300
+	1    0    0    -1
+$EndComp
+Wire Wire Line
+	12200 3150 12150 3150
+Wire Wire Line
+	12150 3150 12150 3250
+Wire Wire Line
+	12200 3250 12150 3250
+Connection ~ 12150 3250
+Wire Wire Line
+	12150 3250 12150 3300
+Wire Wire Line
+	12200 3050 12150 3050
+Wire Wire Line
+	12150 2950 12200 2950
+$Comp
+L MRDT_Connectors:Molex_SL_04 Conn10
+U 1 1 5DE03C76
+P 12400 4050
+F 0 "Conn10" H 12527 4308 60  0000 L CNN
+F 1 "Molex_SL_04" H 12527 4202 60  0000 L CNN
+F 2 "MRDT_Connectors:MOLEX_SL_04_Horizontal" H 12400 4050 60  0001 C CNN
+F 3 "" H 12400 4050 60  0001 C CNN
+	1    12400 4050
+	1    0    0    -1
+$EndComp
+Text GLabel 12150 3700 0    50   Input ~ 0
+ACT_PWR
+Text GLabel 12150 3800 0    50   Input ~ 0
+ACT_PWR
+$Comp
+L power:GND #PWR0114
+U 1 1 5DE03C7E
+P 12150 4050
+F 0 "#PWR0114" H 12150 3800 50  0001 C CNN
+F 1 "GND" H 12155 3877 50  0000 C CNN
+F 2 "" H 12150 4050 50  0001 C CNN
+F 3 "" H 12150 4050 50  0001 C CNN
+	1    12150 4050
+	1    0    0    -1
+$EndComp
+Wire Wire Line
+	12200 3900 12150 3900
+Wire Wire Line
+	12150 3900 12150 4000
+Wire Wire Line
+	12200 4000 12150 4000
+Connection ~ 12150 4000
+Wire Wire Line
+	12150 4000 12150 4050
+Wire Wire Line
+	12200 3800 12150 3800
+Wire Wire Line
+	12150 3700 12200 3700
+$Comp
+L power:GND #PWR0143
+U 1 1 5DE25856
+P 12150 1900
+F 0 "#PWR0143" H 12150 1650 50  0001 C CNN
+F 1 "GND" H 12155 1727 50  0000 C CNN
+F 2 "" H 12150 1900 50  0001 C CNN
+F 3 "" H 12150 1900 50  0001 C CNN
+	1    12150 1900
+	1    0    0    -1
+$EndComp
+Wire Wire Line
+	12150 1750 12200 1750
+Wire Wire Line
+	12150 1900 12150 1850
+Wire Wire Line
+	12150 1850 12200 1850
+$Comp
+L power:+5V #PWR0144
+U 1 1 5DE69DC1
+P 12150 1700
+F 0 "#PWR0144" H 12150 1550 50  0001 C CNN
+F 1 "+5V" H 12165 1873 50  0000 C CNN
+F 2 "" H 12150 1700 50  0001 C CNN
+F 3 "" H 12150 1700 50  0001 C CNN
+	1    12150 1700
+	1    0    0    -1
+$EndComp
+Wire Wire Line
+	12150 1700 12150 1750
+Text Notes 11800 800  0    98   ~ 20
+Extra Outputs
+Text Notes 12200 1450 0    98   ~ 0
+5V
+Text Notes 12150 2750 0    98   ~ 0
+12V
+Wire Notes Line
+	13300 5150 13300 500
+Text Notes 11600 5050 0    50   ~ 0
+Sorry for these 12V connectors. Whole \nandersons for 12V extra busses on a \nmini rover are overkill. But I don't want \nto introduce a new connector outside \nour standards. So two pins on a \nMolex SL will get you 4A.
 $EndSCHEMATC
