File: MiniRoverPowerBoard_Hardware/MiniRoverPowerBoard_Hardware.sch (KiCad schematic (older format))
At the start: 77 parts, among them Q1 Q_NMOS_GSD, Q2 Q_NMOS_GSD, Q3 Q_PMOS_GDS, Q4 Q_NMOS_GSD, SW1 Relay_SPST, SW2 SW_Push, SW3 SW_Push, U1 VNH5019A_E, U2 VNH5019A_E, U3 ACS722xLCTR-40AU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

Commit message: Majority of routing complete; few buses to go
Changed lines of the file:
@@
 Wire Wire Line
 	9250 3800 9600 3800
-Text GLabel 12250 8000 0    50   Output ~ 0
+Text GLabel 12250 8100 0    50   Output ~ 0
 LEFT_PWM
-Text GLabel 12250 8100 0    50   Output ~ 0
+Text GLabel 12250 8400 0    50   Output ~ 0
 RIGHT_PWM
 Wire Wire Line
@@
 Wire Wire Line
 	12300 8100 12250 8100
+Text GLabel 13700 8000 2    50   Input ~ 0
+PACK_IMEAS
 Text GLabel 13700 8100 2    50   Input ~ 0
-PACK_IMEAS
-Text GLabel 13700 8000 2    50   Input ~ 0
 V_LOG_SENSE
 Text GLabel 13700 7900 2    50   Input ~ 0
@@
 Text GLabel 13700 7300 2    50   Input ~ 0
 LOGIC_PWR
-Text GLabel 12250 8200 0    50   Output ~ 0
+Text GLabel 12250 7800 0    50   Output ~ 0
 ESTOP_EN
 Text GLabel 12250 7900 0    50   Output ~ 0
 LOG_SW_EN
+Text GLabel 12250 7700 0    50   Output ~ 0
+BUZZER_EN
+Text GLabel 12250 8700 0    50   Input ~ 0
+LEFT_SW
+Text GLabel 12250 8600 0    50   Input ~ 0
+RIGHT_SW
+Text GLabel 12250 8000 0    50   Output ~ 0
+IN_A1
+Text GLabel 12250 8200 0    50   Output ~ 0
+IN_B1
 Text GLabel 12250 8300 0    50   Output ~ 0
-BUZZER_EN
-Text GLabel 12250 7700 0    50   Input ~ 0
-LEFT_SW
-Text GLabel 12250 7800 0    50   Input ~ 0
-RIGHT_SW
-Text GLabel 12250 8400 0    50   Output ~ 0
-IN_A1
+IN_A2
 Text GLabel 12250 8500 0    50   Output ~ 0
-IN_B1
-Text GLabel 12250 8600 0    50   Output ~ 0
-IN_A2
-Text GLabel 12250 8700 0    50   Output ~ 0
 IN_B2
 $Comp

Commit message: Layout & silkscreen complete; Ready for review
Changed lines of the file:
@@
 Wire Wire Line
 	12300 8100 12250 8100
-Text GLabel 13700 8000 2    50   Input ~ 0
+Text GLabel 13700 7900 2    50   Input ~ 0
 PACK_IMEAS
 Text GLabel 13700 8100 2    50   Input ~ 0
 V_LOG_SENSE
-Text GLabel 13700 7900 2    50   Input ~ 0
+Text GLabel 13700 8000 2    50   Input ~ 0
 V_ACT_SENSE
 Text GLabel 13700 7300 2    50   Input ~ 0

Commit message: Removed 3v3 AP1509 and changed voltage dividers
Parts:
- removed C3, C7: 10u, Capacitor_SMD:C_0603_1608Metric_Pad1.05x0.95mm_HandSolder, symbol Device:C_Small
- removed Conn7: Molex_SL_02, MRDT_Connectors:MOLEX_SL_02_Vertical, symbol MRDT_Connectors:Molex_SL_02
- removed D7: D_Schottky, Diode_SMD:D_0603_1608Metric_Pad1.05x0.95mm_HandSolder, symbol Device:D_Schottky_Small
- removed L1: 47uH, Capacitor_THT:CP_Radial_D5.0mm_P2.00mm, symbol pspice:INDUCTOR
- removed R15, R26, R27: 0, Resistor_SMD:R_0603_1608Metric_Pad1.05x0.95mm_HandSolder, symbol Device:R_Small
- removed U4: AP1509, Package_SO:SOIC-8_3.9x4.9mm_P1.27mm, symbol MRDT_ICs:AP1509
- added Conn7: Molex_SL_03, symbol MRDT_Connectors:Molex_SL_03
- D1, D9: value 3V3_Zener -> 4.7V_Zener
- F1: value 30A_Fuse -> 35A_Fuse
- R22, R8: value 20k -> 21k
- R23, R9: value 13k -> 26.7k
Connections:
- wire segments 371 -> 333
- no-connect marks 14 -> 13
Other:
- note added: "8.4V to 4.7V"
- note added: "Min Input Volatge: 7V"
- note added: "Min Input Voltage: 4.5V\n500mA limit due to inductor"
- note removed: "3V3 Regulation"
- note removed: "8.4V to 3.3V"
- note removed: "Min Input Volatge: 6V"
- note removed: "Min Input Voltage for each: 4.5V\n500mA limit each due to inductors"

Commit message: Finished board changes for arduino pwr & added gerbs
Parts:
- added R15, R26: 0, Resistor_SMD:R_0603_1608Metric_Pad1.05x0.95mm_HandSolder, symbol Device:R_Small
- Conn10, Conn9: footprint MRDT_Connectors:MOLEX_SL_04_Horizontal -> MRDT_Connectors:MOLEX_SL_04_Vertical
- Conn7: footprint (none) -> MRDT_Connectors:MOLEX_SL_03_Vertical
Connections:
- net labels added: 5V_R, VIN_R
- wire segments 333 -> 336
- no-connect marks 13 -> 12
Changed lines of the file:
@@
 Text GLabel 13700 8000 2    50   Input ~ 0
 V_ACT_SENSE
-Text GLabel 13700 7300 2    50   Input ~ 0
+Text GLabel 14300 7300 2    50   Input ~ 0
 LOGIC_PWR
 Text GLabel 12250 7800 0    50   Output ~ 0
@@
 	13700 7400 13650 7400
 Wire Wire Line
-	13650 7300 13700 7300
-Wire Wire Line
 	13650 8100 13700 8100
 Wire Wire Line
@@
 Wire Notes Line
 	7600 6750 10300 6750
-Text Notes 14250 7350 0    50   ~ 0
+Text Notes 14300 6950 0    50   ~ 0
 Min Input Volatge: 7V
 NoConn ~ 13650 7200
 NoConn ~ 13650 7100
 NoConn ~ 13650 7500
-NoConn ~ 13650 7600
 NoConn ~ 12300 7500
 NoConn ~ 12300 7200
@@
 F 0 "Conn9" H 12527 3558 60  0000 L CNN
 F 1 "Molex_SL_04" H 12527 3452 60  0000 L CNN
-F 2 "MRDT_Connectors:MOLEX_SL_04_Horizontal" H 12400 3300 60  0001 C CNN
+F 2 "MRDT_Connectors:MOLEX_SL_04_Vertical" H 12400 3300 60  0001 C CNN
 F 3 "" H 12400 3300 60  0001 C CNN
 	1    12400 3300
@@
 F 0 "Conn10" H 12527 4308 60  0000 L CNN
 F 1 "Molex_SL_04" H 12527 4202 60  0000 L CNN
-F 2 "MRDT_Connectors:MOLEX_SL_04_Horizontal" H 12400 4050 60  0001 C CNN
+F 2 "MRDT_Connectors:MOLEX_SL_04_Vertical" H 12400 4050 60  0001 C CNN
 F 3 "" H 12400 4050 60  0001 C CNN
 	1    12400 4050
@@
 Sorry for these 12V connectors. Whole \nandersons for 12V extra busses on a \nmini rover are overkill. But I don't want \nto introduce a new connector outside \nour standards. So two pins on a \nMolex SL will get you 4A.
 $Comp
-L power:+3V3 #PWR?
+L power:+3V3 #PWR0133
 U 1 1 5DF504B1
 P 13700 8600
-F 0 "#PWR?" H 13700 8450 50  0001 C CNN
+F 0 "#PWR0133" H 13700 8450 50  0001 C CNN
 F 1 "+3V3" V 13700 8800 50  0000 C CNN
 F 2 "" H 13700 8600 50  0001 C CNN
@@
 F 0 "Conn7" H 6577 6208 60  0000 L CNN
 F 1 "Molex_SL_03" H 6577 6102 60  0000 L CNN
-F 2 "" H 6450 6000 60  0001 C CNN
+F 2 "MRDT_Connectors:MOLEX_SL_03_Vertical" H 6450 6000 60  0001 C CNN
 F 3 "" H 6450 6000 60  0001 C CNN
 	1    6450 6000
@@
 $EndComp
 $Comp
-L power:GND #PWR?
+L power:GND #PWR0134
 U 1 1 5E047F67
 P 6200 6000
-F 0 "#PWR?" H 6200 5750 50  0001 C CNN
+F 0 "#PWR0134" H 6200 5750 50  0001 C CNN
 F 1 "GND" H 6205 5827 50  0000 C CNN
 F 2 "" H 6200 6000 50  0001 C CNN
@@
 Wire Wire Line
 	6200 5950 6250 5950
+$Comp
+L power:+5V #PWR0145
+U 1 1 5DF5E744
+P 14300 7600
+F 0 "#PWR0145" H 14300 7450 50  0001 C CNN
+F 1 "+5V" H 14315 7773 50  0000 C CNN
+F 2 "" H 14300 7600 50  0001 C CNN
+F 3 "" H 14300 7600 50  0001 C CNN
+	1    14300 7600
+	0    1    1    0
+$EndComp
+$Comp
+L Device:R_Small R15
+U 1 1 5DF82801
+P 14150 7300
+F 0 "R15" V 14250 7250 50  0000 L CNN
+F 1 "0" V 14150 7300 50  0000 C CNN
+F 2 "Resistor_SMD:R_0603_1608Metric_Pad1.05x0.95mm_HandSolder" H 14150 7300 50  0001 C CNN
+F 3 "ERJ-PB3B2102V" H 14150 7300 50  0001 C CNN
+	1    14150 7300
+	0    -1   -1   0
+$EndComp
+$Comp
+L Device:R_Small R26
+U 1 1 5DF83E9F
+P 14150 7600
+F 0 "R26" V 14250 7550 50  0000 L CNN
+F 1 "0" V 14150 7600 50  0000 C CNN
+F 2 "Resistor_SMD:R_0603_1608Metric_Pad1.05x0.95mm_HandSolder" H 14150 7600 50  0001 C CNN
+F 3 "ERJ-PB3B2102V" H 14150 7600 50  0001 C CNN
+	1    14150 7600
+	0    -1   -1   0
+$EndComp
+Wire Wire Line
+	14250 7600 14300 7600
+Wire Wire Line
+	14250 7300 14300 7300
+Wire Wire Line
+	14050 7300 13650 7300
+Wire Wire Line
+	13650 7600 14050 7600
+Text Label 13700 7300 0    50   ~ 0
+VIN_R
+Text Label 13700 7600 0    50   ~ 0
+5V_R
 $EndSCHEMATC
